File: hardware/kicad_docs/whooshy_sound.kicad_pcb (KiCad board)
At the start: 4 copper layers, 83.8 x 80 mm, 115 parts, among them J1 audio_in, J10 SWD_header, J2 audio_out, J3 extern_cutoff_CV_TRS, J4 extern_rez_CV_TRS, J5 9VDC_in, J6 signal_in, J7 signal_out, J8 cutoff_CV_in, J9 rez_CV_and_PS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

Commit message: tweak pcb
Routing:
- net -12V: track 175.3 -> 185.6 mm
- net Net-(C28-Pad1): track 61.2 -> 55.7 mm
- net /cutoff_CV_generator/summed_cutoff_CV_out: track 66.5 -> 67.8 mm
- net -5V: track 102.6 -> 103.3 mm
- net GND: track 6.13 -> 6.38 mm, vias 25 -> 39
