File: hardware/front_panel/kicad_docs/whooshy_sound_front_panel.kicad_pcb (KiCad board)
At the start: 2 copper layers, 86.4 x 101.6 mm, 4 parts

Commit message: add LED driver, change LED to 5mm
Other:
- outline, holes or cut-outs redrawn
Changed lines of the file:
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@@
       (effects (font (size 1 1) (thickness 0.15)))
     )
+    (fp_circle (center 0 0) (end 3.45 0) (layer F.CrtYd) (width 0.05))
     (fp_circle (center 0 0) (end 3.2 0) (layer Cmts.User) (width 0.15))
-    (fp_circle (center 0 0) (end 3.45 0) (layer F.CrtYd) (width 0.05))
     (fp_text user %R (at 0.3 0) (layer F.Fab)
       (effects (font (size 1 1) (thickness 0.15)))
@@
       (effects (font (size 1 1) (thickness 0.15)))
     )
+    (fp_circle (center 0 0) (end 3.45 0) (layer F.CrtYd) (width 0.05))
     (fp_circle (center 0 0) (end 3.2 0) (layer Cmts.User) (width 0.15))
-    (fp_circle (center 0 0) (end 3.45 0) (layer F.CrtYd) (width 0.05))
     (fp_text user %R (at 0.3 0) (layer F.Fab)
       (effects (font (size 1 1) (thickness 0.15)))
@@
       (effects (font (size 1 1) (thickness 0.15)))
     )
+    (fp_circle (center 0 0) (end 3.45 0) (layer F.CrtYd) (width 0.05))
     (fp_circle (center 0 0) (end 3.2 0) (layer Cmts.User) (width 0.15))
-    (fp_circle (center 0 0) (end 3.45 0) (layer F.CrtYd) (width 0.05))
     (fp_text user %R (at 0.3 0) (layer F.Fab)
       (effects (font (size 1 1) (thickness 0.15)))
@@
       (effects (font (size 1 1) (thickness 0.15)))
     )
+    (fp_circle (center 0 0) (end 3.45 0) (layer F.CrtYd) (width 0.05))
     (fp_circle (center 0 0) (end 3.2 0) (layer Cmts.User) (width 0.15))
-    (fp_circle (center 0 0) (end 3.45 0) (layer F.CrtYd) (width 0.05))
     (fp_text user %R (at 0.3 0) (layer F.Fab)
       (effects (font (size 1 1) (thickness 0.15)))
@@
   (gr_line (start 74.295 23.495) (end 159.385 23.495) (layer Dwgs.User) (width 0.15))
   (gr_circle (center 116.84 127) (end 126.84 127) (layer Dwgs.User) (width 0.15))
-  (gr_circle (center 101.6 127) (end 103.15 127) (layer Edge.Cuts) (width 0.05))
+  (gr_circle (center 101.6 127) (end 104.15 127) (layer Edge.Cuts) (width 0.05))
   (gr_circle (center 116.84 127) (end 121.64 127) (layer Edge.Cuts) (width 0.05))
   (gr_text norm. (at 146.05 95.25) (layer F.SilkS)
