File: hardware/main_pcb/kicad_docs/power_supply.sch (KiCad schematic (older format))
At the start: 47 parts, among them U1 TL072, U2 LM4040DBZ-5, U3 LT3467A, U4 LT1117-3.3, U5 TL072, U6 TL072, U7 TL072

Commit message: move main pcb into its own dir
Parts:
- added D8: LED, LED_THT:LED_D3.0mm, symbol Device:LED
- added J11: LED_switch, Connector_PinHeader_2.54mm:PinHeader_1x02_P2.54mm_Vertical, symbol Connector_Generic:Conn_01x02
- added R37: 2k2, Resistor_SMD:R_0805_2012Metric, symbol Device:R
- R5: value R -> 2k2
Connections:
- net +9V: now also R37.1; no longer FB4.2
- net -12V: now also FB4.1
- net GND: now also C13.1, C14.1, U2.1 (K), D8.1 (K); no longer C13.2, R5.2
- new net: J11.1 (Pin_1), R37.2
- new net: D8.2 (A), J11.2 (Pin_2)
- new net: C13.2, FB4.2, R5.2
Other:
- note added: "Status LED"
- moved on the sheet: C13, C14, FB4, R5, U2
Changed lines of the file:
@@
 L Reference_Voltage:LM4040DBZ-5 U2
 U 1 1 61358642
-P 9350 1750
-F 0 "U2" V 9396 1662 50  0000 R CNN
-F 1 "LM4040DBZ-5" V 9305 1662 50  0000 R CNN
-F 2 "Package_TO_SOT_SMD:SOT-23" H 9350 1550 50  0001 C CIN
-F 3 "http://www.ti.com/lit/ds/symlink/lm4040-n.pdf" H 9350 1750 50  0001 C CIN
-	1    9350 1750
+P 9500 1300
+F 0 "U2" V 9546 1212 50  0000 R CNN
+F 1 "LM4040DBZ-5" V 9455 1212 50  0000 R CNN
+F 2 "Package_TO_SOT_SMD:SOT-23" H 9500 1100 50  0001 C CIN
+F 3 "http://www.ti.com/lit/ds/symlink/lm4040-n.pdf" H 9500 1300 50  0001 C CIN
+	1    9500 1300
 	0    -1   -1   0
 $EndComp
@@
 L power:-5V #PWR020
 U 1 1 6135B225
-P 10250 2200
-F 0 "#PWR020" H 10250 2300 50  0001 C CNN
-F 1 "-5V" H 10265 2373 50  0000 C CNN
-F 2 "" H 10250 2200 50  0001 C CNN
-F 3 "" H 10250 2200 50  0001 C CNN
-	1    10250 2200
+P 10400 1750
+F 0 "#PWR020" H 10400 1850 50  0001 C CNN
+F 1 "-5V" H 10415 1923 50  0000 C CNN
+F 2 "" H 10400 1750 50  0001 C CNN
+F 3 "" H 10400 1750 50  0001 C CNN
+	1    10400 1750
 	-1   0    0    1
 $EndComp
@@
 L Device:R R5
 U 1 1 61365218
-P 9350 2250
-F 0 "R5" H 9420 2296 50  0000 L CNN
-F 1 "R" H 9420 2205 50  0000 L CNN
-F 2 "Resistor_SMD:R_0805_2012Metric" V 9280 2250 50  0001 C CNN
-F 3 "~" H 9350 2250 50  0001 C CNN
-	1    9350 2250
+P 9500 1800
+F 0 "R5" H 9570 1846 50  0000 L CNN
+F 1 "2k2" H 9570 1755 50  0000 L CNN
+F 2 "Resistor_SMD:R_0805_2012Metric" V 9430 1800 50  0001 C CNN
+F 3 "~" H 9500 1800 50  0001 C CNN
+	1    9500 1800
 	1    0    0    -1
 $EndComp
@@
 L Device:C C13
 U 1 1 61365860
-P 8750 2000
-F 0 "C13" H 8865 2046 50  0000 L CNN
-F 1 "100n" H 8865 1955 50  0000 L CNN
-F 2 "Capacitor_SMD:C_0805_2012Metric" H 8788 1850 50  0001 C CNN
-F 3 "~" H 8750 2000 50  0001 C CNN
-	1    8750 2000
+P 8900 1550
+F 0 "C13" H 9015 1596 50  0000 L CNN
+F 1 "100n" H 9015 1505 50  0000 L CNN
+F 2 "Capacitor_SMD:C_0805_2012Metric" H 8938 1400 50  0001 C CNN
+F 3 "~" H 8900 1550 50  0001 C CNN
+	1    8900 1550
 	1    0    0    -1
 $EndComp
@@
 L Device:C C14
 U 1 1 61365E02
-P 10250 1750
-F 0 "C14" H 10365 1796 50  0000 L CNN
-F 1 "100n" H 10365 1705 50  0000 L CNN
-F 2 "Capacitor_SMD:C_0805_2012Metric" H 10288 1600 50  0001 C CNN
-F 3 "~" H 10250 1750 50  0001 C CNN
-	1    10250 1750
-	1    0    0    -1
-$EndComp
-Wire Wire Line
-	8750 1850 8750 1450
-Wire Wire Line
-	8750 1450 9200 1450
-Wire Wire Line
-	9350 1450 9350 1600
-Wire Wire Line
-	9350 2400 9350 2550
-Wire Wire Line
-	9350 2550 8750 2550
-Wire Wire Line
-	8750 2550 8750 2150
-Wire Wire Line
-	9350 1900 9350 2000
-Wire Wire Line
-	9350 2000 10250 2000
-Wire Wire Line
-	10250 2000 10250 1900
-Connection ~ 9350 2000
-Wire Wire Line
-	9350 2000 9350 2100
-Wire Wire Line
-	10250 1600 10250 1450
-Wire Wire Line
-	10250 1450 9350 1450
-Connection ~ 9350 1450
-Wire Wire Line
-	10250 2200 10250 2100
-Connection ~ 10250 2000
-$Comp
-L power:GND #PWR019
-U 1 1 61369B5F
-P 9350 2650
-F 0 "#PWR019" H 9350 2400 50  0001 C CNN
-F 1 "GND" H 9355 2477 50  0000 C CNN
-F 2 "" H 9350 2650 50  0001 C CNN
-F 3 "" H 9350 2650 50  0001 C CNN
-	1    9350 2650
-	1    0    0    -1
-$EndComp
-Wire Wire Line
-	9350 2650 9350 2550
-Connection ~ 9350 2550
-$Comp
-L power:+9V #PWR018
-U 1 1 6136B01B
-P 9200 1150
-F 0 "#PWR018" H 9200 1000 50  0001 C CNN
-F 1 "+9V" H 9215 1323 50  0000 C CNN
-F 2 "" H 9200 1150 50  0001 C CNN
-F 3 "" H 9200 1150 50  0001 C CNN
-	1    9200 1150
-	1    0    0    -1
-$EndComp
-Wire Wire Line
-	9200 1350 9200 1450
-Connection ~ 9200 1450
-Wire Wire Line
-	9200 1450 9350 1450
+P 10400 1300
+F 0 "C14" H 10515 1346 50  0000 L CNN
+F 1 "100n" H 10515 1255 50  0000 L CNN
+F 2 "Capacitor_SMD:C_0805_2012Metric" H 10438 1150 50  0001 C CNN
+F 3 "~" H 10400 1300 50  0001 C CNN
+	1    10400 1300
+	1    0    0    -1
+$EndComp
+Wire Wire Line
+	8900 1400 8900 1000
+Wire Wire Line
+	9500 1000 9500 1150
+Wire Wire Line
+	9500 1950 9500 2100
+Wire Wire Line
+	9500 2100 8900 2100
+Wire Wire Line
+	8900 2100 8900 1700
+Wire Wire Line
+	9500 1450 9500 1550
+Wire Wire Line
+	9500 1550 10400 1550
+Wire Wire Line
+	10400 1550 10400 1450
+Connection ~ 9500 1550
+Wire Wire Line
+	9500 1550 9500 1650
+Wire Wire Line
+	10400 1150 10400 1000
+Wire Wire Line
+	10400 1000 9500 1000
+Connection ~ 9500 1000
+Wire Wire Line
+	10400 1750 10400 1650
+Connection ~ 10400 1550
+Wire Wire Line
+	9500 2200 9500 2100
+Connection ~ 9500 2100
 $Comp
 L Device:Ferrite_Bead_Small FB2
@@
 L Device:Ferrite_Bead_Small FB4
 U 1 1 6143CF7E
-P 9200 1250
-F 0 "FB4" H 9100 1204 50  0000 R CNN
-F 1 "100R @ 100MHz" H 9100 1295 50  0000 R CNN
-F 2 "Inductor_SMD:L_0805_2012Metric" V 9130 1250 50  0001 C CNN
-F 3 "~" H 9200 1250 50  0001 C CNN
-	1    9200 1250
+P 9500 2300
+F 0 "FB4" H 9400 2254 50  0000 R CNN
+F 1 "100R @ 100MHz" H 9400 2345 50  0000 R CNN
+F 2 "Inductor_SMD:L_0805_2012Metric" V 9430 2300 50  0001 C CNN
+F 3 "~" H 9500 2300 50  0001 C CNN
+	1    9500 2300
 	-1   0    0    1
 $EndComp
@@
 L power:PWR_FLAG #FLG01
 U 1 1 60D2E894
-P 10600 2200
-F 0 "#FLG01" H 10600 2275 50  0001 C CNN
-F 1 "PWR_FLAG" H 10600 2373 50  0000 C CNN
-F 2 "" H 10600 2200 50  0001 C CNN
-F 3 "~" H 10600 2200 50  0001 C CNN
-	1    10600 2200
+P 10750 1750
+F 0 "#FLG01" H 10750 1825 50  0001 C CNN
+F 1 "PWR_FLAG" H 10750 1923 50  0000 C CNN
+F 2 "" H 10750 1750 50  0001 C CNN
+F 3 "~" H 10750 1750 50  0001 C CNN
+	1    10750 1750
 	-1   0    0    1
 $EndComp
 Wire Wire Line
-	10250 2100 10600 2100
-Connection ~ 10250 2100
-Wire Wire Line
-	10250 2100 10250 2000
+	10400 1650 10750 1650
+Connection ~ 10400 1650
+Wire Wire Line
+	10400 1650 10400 1550
 $Comp
 L power:PWR_FLAG #FLG05
@@
 	8750 6150 8750 5950
 Wire Wire Line
-	10600 2200 10600 2100
+	10750 1750 10750 1650
 Text Notes 8750 850  0    118  ~ 0
 -5 volt reference
@@
 	2050 1600 1100 1600
 Connection ~ 2050 1600
+$Comp
+L Device:R R37
+U 1 1 60CE0C59
+P 5650 6800
+F 0 "R37" H 5720 6846 50  0000 L CNN
+F 1 "2k2" H 5720 6755 50  0000 L CNN
+F 2 "Resistor_SMD:R_0805_2012Metric" V 5580 6800 50  0001 C CNN
+F 3 "~" H 5650 6800 50  0001 C CNN
+	1    5650 6800
+	1    0    0    -1
+$EndComp
+$Comp
+L Device:LED D8
+U 1 1 60CE18AF
+P 5650 7450
+F 0 "D8" V 5689 7332 50  0000 R CNN
+F 1 "LED" V 5598 7332 50  0000 R CNN
+F 2 "LED_THT:LED_D3.0mm" H 5650 7450 50  0001 C CNN
+F 3 "~" H 5650 7450 50  0001 C CNN
+	1    5650 7450
+	0    -1   -1   0
+$EndComp
+$Comp
+L Connector_Generic:Conn_01x02 J11
+U 1 1 60CEEAB6
+P 5250 7100
+F 0 "J11" H 5168 7317 50  0000 C CNN
+F 1 "LED_switch" H 5168 7226 50  0000 C CNN
+F 2 "Connector_PinHeader_2.54mm:PinHeader_1x02_P2.54mm_Vertical" H 5250 7100 50  0001 C CNN
+F 3 "~" H 5250 7100 50  0001 C CNN
+	1    5250 7100
+	-1   0    0    -1
+$EndComp
+$Comp
+L power:+9V #PWR069
+U 1 1 60CF2A5B
+P 5650 6650
+F 0 "#PWR069" H 5650 6500 50  0001 C CNN
+F 1 "+9V" H 5665 6823 50  0000 C CNN
+F 2 "" H 5650 6650 50  0001 C CNN
+F 3 "" H 5650 6650 50  0001 C CNN
+	1    5650 6650
+	1    0    0    -1
+$EndComp
+$Comp
+L power:GND #PWR070
+U 1 1 60CFFFB7
+P 5650 7600
+F 0 "#PWR070" H 5650 7350 50  0001 C CNN
+F 1 "GND" H 5655 7427 50  0000 C CNN
+F 2 "" H 5650 7600 50  0001 C CNN
+F 3 "" H 5650 7600 50  0001 C CNN
+	1    5650 7600
+	1    0    0    -1
+$EndComp
+Text Notes 5100 6400 0    118  ~ 0
+Status LED
+Wire Wire Line
+	5650 7300 5650 7200
+Wire Wire Line
+	5650 7200 5450 7200
+Wire Wire Line
+	5450 7100 5650 7100
+Wire Wire Line
+	5650 7100 5650 6950
+Wire Wire Line
+	8900 1000 9500 1000
+$Comp
+L power:GND #PWR?
+U 1 1 60E3D478
+P 8600 1200
+F 0 "#PWR?" H 8600 950 50  0001 C CNN
+F 1 "GND" H 8605 1027 50  0000 C CNN
+F 2 "" H 8600 1200 50  0001 C CNN
+F 3 "" H 8600 1200 50  0001 C CNN
+	1    8600 1200
+	1    0    0    -1
+$EndComp
+Wire Wire Line
+	8600 1200 8600 1000
+Wire Wire Line
+	8600 1000 8900 1000
+Connection ~ 8900 1000
+$Comp
+L power:-12V #PWR?
+U 1 1 60E4AA03
+P 9500 2400
+F 0 "#PWR?" H 9500 2500 50  0001 C CNN
+F 1 "-12V" H 9515 2573 50  0000 C CNN
+F 2 "" H 9500 2400 50  0001 C CNN
+F 3 "" H 9500 2400 50  0001 C CNN
+	1    9500 2400
+	-1   0    0    1
+$EndComp
 $EndSCHEMATC

Commit message: add LED driver, change LED to 5mm
Parts:
- removed D8: LED, LED_THT:LED_D3.0mm, symbol Device:LED
- removed J11: LED_switch, Connector_PinHeader_2.54mm:PinHeader_1x02_P2.54mm_Vertical, symbol Connector_Generic:Conn_01x02
- removed R37: 2k2, Resistor_SMD:R_0805_2012Metric, symbol Device:R
Other:
- note removed: "Status LED"
Changed lines of the file:
@@
 	2050 1600 1100 1600
 Connection ~ 2050 1600
-$Comp
-L Device:R R37
-U 1 1 60CE0C59
-P 5650 6800
-F 0 "R37" H 5720 6846 50  0000 L CNN
-F 1 "2k2" H 5720 6755 50  0000 L CNN
-F 2 "Resistor_SMD:R_0805_2012Metric" V 5580 6800 50  0001 C CNN
-F 3 "~" H 5650 6800 50  0001 C CNN
-	1    5650 6800
-	1    0    0    -1
-$EndComp
-$Comp
-L Device:LED D8
-U 1 1 60CE18AF
-P 5650 7450
-F 0 "D8" V 5689 7332 50  0000 R CNN
-F 1 "LED" V 5598 7332 50  0000 R CNN
-F 2 "LED_THT:LED_D3.0mm" H 5650 7450 50  0001 C CNN
-F 3 "~" H 5650 7450 50  0001 C CNN
-	1    5650 7450
-	0    -1   -1   0
-$EndComp
-$Comp
-L Connector_Generic:Conn_01x02 J11
-U 1 1 60CEEAB6
-P 5250 7100
-F 0 "J11" H 5168 7317 50  0000 C CNN
-F 1 "LED_switch" H 5168 7226 50  0000 C CNN
-F 2 "Connector_PinHeader_2.54mm:PinHeader_1x02_P2.54mm_Vertical" H 5250 7100 50  0001 C CNN
-F 3 "~" H 5250 7100 50  0001 C CNN
-	1    5250 7100
-	-1   0    0    -1
-$EndComp
-$Comp
-L power:+9V #PWR069
-U 1 1 60CF2A5B
-P 5650 6650
-F 0 "#PWR069" H 5650 6500 50  0001 C CNN
-F 1 "+9V" H 5665 6823 50  0000 C CNN
-F 2 "" H 5650 6650 50  0001 C CNN
-F 3 "" H 5650 6650 50  0001 C CNN
-	1    5650 6650
-	1    0    0    -1
-$EndComp
-$Comp
-L power:GND #PWR070
-U 1 1 60CFFFB7
-P 5650 7600
-F 0 "#PWR070" H 5650 7350 50  0001 C CNN
-F 1 "GND" H 5655 7427 50  0000 C CNN
-F 2 "" H 5650 7600 50  0001 C CNN
-F 3 "" H 5650 7600 50  0001 C CNN
-	1    5650 7600
-	1    0    0    -1
-$EndComp
-Text Notes 5100 6400 0    118  ~ 0
-Status LED
-Wire Wire Line
-	5650 7300 5650 7200
-Wire Wire Line
-	5650 7200 5450 7200
-Wire Wire Line
-	5450 7100 5650 7100
-Wire Wire Line
-	5650 7100 5650 6950
 Wire Wire Line
 	8900 1000 9500 1000
 $Comp
-L power:GND #PWR?
+L power:GND #PWR018
 U 1 1 60E3D478
 P 8600 1200
-F 0 "#PWR?" H 8600 950 50  0001 C CNN
+F 0 "#PWR018" H 8600 950 50  0001 C CNN
 F 1 "GND" H 8605 1027 50  0000 C CNN
 F 2 "" H 8600 1200 50  0001 C CNN
@@
 Connection ~ 8900 1000
 $Comp
-L power:-12V #PWR?
+L power:-12V #PWR019
 U 1 1 60E4AA03
 P 9500 2400
-F 0 "#PWR?" H 9500 2500 50  0001 C CNN
+F 0 "#PWR019" H 9500 2500 50  0001 C CNN
 F 1 "-12V" H 9515 2573 50  0000 C CNN
 F 2 "" H 9500 2400 50  0001 C CNN

Commit message: flip env invert switch, condense cap types
Parts:
- C25: value 2u2 -> 10u
- C6: value 10n -> 100n
- C8: value 47n -> 100n
Changed lines of the file:
@@
 P 5250 4750
 F 0 "C8" H 5365 4796 50  0000 L CNN
-F 1 "47n" H 5365 4705 50  0000 L CNN
+F 1 "100n" H 5365 4705 50  0000 L CNN
 F 2 "Capacitor_SMD:C_0805_2012Metric" H 5288 4600 50  0001 C CNN
 F 3 "~" H 5250 4750 50  0001 C CNN
@@
 P 7400 1600
 F 0 "C6" H 7515 1646 50  0000 L CNN
-F 1 "10n" H 7515 1555 50  0000 L CNN
+F 1 "100n" H 7515 1555 50  0000 L CNN
 F 2 "Capacitor_SMD:C_0805_2012Metric" H 7438 1450 50  0001 C CNN
 F 3 "~" H 7400 1600 50  0001 C CNN
@@
 P 3000 7150
 F 0 "C25" H 3115 7196 50  0000 L CNN
-F 1 "2u2" H 3115 7105 50  0000 L CNN
+F 1 "10u" H 3115 7105 50  0000 L CNN
 F 2 "Capacitor_SMD:C_0805_2012Metric" H 3038 7000 50  0001 C CNN
 F 3 "~" H 3000 7150 50  0001 C CNN
